File: PCB/_restore_backup_2026-09-26T18-27-32-307/praevius.kicad_pcb (KiCad board)
At the start: 2 copper layers, 33 parts

Commit message: Working on MCU footprint
Parts:
- removed the REF** at (283.1, 81.6)
- removed the REF** at (283.1, 76.5)
- removed the REF** at (283.1, 89.1)
- removed the REF** at (283.1, 84.1)
- removed the REF** at (283.1, 79.0)
- removed the REF** at (283.2, 66.3)
- removed the REF** at (283.2, 68.9)
- removed the REF** at (283.1, 91.7)
- removed the REF** at (283.1, 74.0)
- removed the REF** at (283.2, 63.8)
- removed the REF** at (283.1, 86.6)
- added REF**: XIAO-nRF52840-Plus-SMD, Seeed Studio XIAO Series Library:XIAO-nRF52840-Plus-SMD, F.Cu at (258.5, 83.5)
- moved REF** 140.6 mm to (210.0, 191.5)
