File: PCB/praevius.kicad_pcb (KiCad board)
At the start: 2 copper layers, 33 parts

Commit message: journal edit
Parts:
- removed REF** (x12): SolderJumper-2_P1.3mm_Open_TrianglePad1.0x1.5mm, Jumper:SolderJumper-2_P1.3mm_Open_TrianglePad1.0x1.5mm
- moved S19 195.8 mm to (74.2, 6.84)
- moved S20 195.6 mm to (94.3, 8.97)
- moved S14 195.4 mm to (76.4, -34.1)
- moved S17 195.4 mm to (95.4, -33.8)
- moved S2 195.4 mm to (-1.66, -18.9)
- moved S8 195.4 mm to (37.0, -32.8)
- moved S7 195.4 mm to (37.7, -13.8)
- moved S5 195.4 mm to (17.3, -20.6)
- moved S12 195.4 mm to (55.2, -57.2)
- moved S11 195.4 mm to (55.9, -38.2)
- moved S13 195.4 mm to (76.1, -15.1)
- moved S1 195.4 mm to (0.00, 0.00)
- moved S15 195.4 mm to (76.7, -53.1)
- moved S18 195.4 mm to (95.7, -52.8)
- moved S10 195.4 mm to (56.5, -19.2)
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Other:
- net class Default added: clearance 0.2, trace_width 0.25, via_dia 0.8, via_drill 0.4

Commit message: Started schematic
Parts:
- removed the S1 at (0.00, 0.00)
- removed the S10 at (56.5, -19.2)
- removed the S11 at (55.9, -38.2)
- removed the S12 at (55.2, -57.2)
- removed the S13 at (76.1, -15.1)
- removed the S14 at (76.4, -34.1)
- removed the S15 at (76.7, -53.1)
- removed the S16 at (95.1, -14.8)
- removed the S17 at (95.4, -33.8)
- removed the S18 at (95.7, -52.8)
- removed the S19 at (74.2, 6.84)
- removed the S2 at (-1.66, -18.9)
- removed the S20 at (94.3, 8.97)
- removed the S21 at (114.2, 15.3)
- removed the S3 at (-3.31, -37.9)
- removed the S4 at (18.9, -1.66)
- removed the S5 at (17.3, -20.6)
- removed the S6 at (15.6, -39.5)
- removed the S7 at (37.7, -13.8)
- removed the S8 at (37.0, -32.8)
- removed the S9 at (36.4, -51.8)
- added REF**: XIAO-nRF52840-Plus-SMD, keeb-footprints:XIAO-nRF52840-Plus-SMD, F.Cu at (75.5, 104.0)
- added S1: , MX, F.Cu at (60.4, 156.7)
- added S1: , MX, B.Cu at (349.3, 159.7)
- added S10: , MX, F.Cu at (117.0, 137.5)
- added S10: , MX, B.Cu at (292.8, 140.5)
- added S11: , MX, F.Cu at (116.3, 118.6)
- added S11: , MX, B.Cu at (293.4, 121.5)
- added S12: , MX, F.Cu at (115.6, 99.6)
- added S12: , MX, B.Cu at (294.1, 102.5)
- added S13: , MX, F.Cu at (136.6, 141.6)
- added S13: , MX, B.Cu at (273.1, 144.5)
- added S14: , MX, F.Cu at (136.9, 122.6)
- added S14: , MX, B.Cu at (272.8, 125.5)
- added S15: , MX, F.Cu at (137.3, 103.6)
- added S15: , MX, B.Cu at (272.5, 106.5)
- added S16: , MX, F.Cu at (155.6, 141.9)
- added S16: , MX, B.Cu at (254.1, 144.9)
- added S17: , MX, F.Cu at (155.9, 122.9)
- added S17: , MX, B.Cu at (253.8, 125.9)
- added S18: , MX, F.Cu at (156.3, 103.9)
- added S18: , MX, B.Cu at (253.5, 106.9)
- added S19: , MX, F.Cu at (134.7, 163.6)
- added S19: , MX, B.Cu at (275.0, 166.5)
- added S2: , MX, F.Cu at (58.8, 137.8)
- added S2: , MX, B.Cu at (350.9, 140.7)
- added S20: , MX, F.Cu at (155.3, 165.6)
- added S20: , MX, B.Cu at (254.4, 168.5)
- added S21: , MX, F.Cu at (175.7, 172.0)
- added S21: , MX, B.Cu at (234.1, 175.0)
- added S3: , MX, F.Cu at (57.1, 118.9)
- added S3: , MX, B.Cu at (352.6, 121.8)
- added S4: , MX, F.Cu at (79.4, 155.1)
- added S4: , MX, B.Cu at (330.4, 158.0)
- added S5: , MX, F.Cu at (77.7, 136.2)
- added S5: , MX, B.Cu at (332.0, 139.1)
- added S6: , MX, F.Cu at (76.1, 117.2)
- added S6: , MX, B.Cu at (333.7, 120.2)
- added S7: , MX, F.Cu at (98.1, 142.9)
- added S7: , MX, B.Cu at (311.6, 145.9)
- added S8: , MX, F.Cu at (97.5, 124.0)
- added S8: , MX, B.Cu at (312.2, 126.9)
- added S9: , MX, F.Cu at (96.8, 105.0)
- added S9: , MX, B.Cu at (312.9, 107.9)
Other:
- net class Default removed

Commit message: Made switch footprints, decided on battery and MCU position
Parts:
- removed the S1 at (60.4, 156.7)
- removed the S1 at (349.3, 159.7)
- removed the S10 at (117.0, 137.5)
- removed the S10 at (292.8, 140.5)
- removed the S11 at (116.3, 118.6)
- removed the S11 at (293.4, 121.5)
- removed the S12 at (115.6, 99.6)
- removed the S12 at (294.1, 102.5)
- removed the S13 at (136.6, 141.6)
- removed the S13 at (273.1, 144.5)
- removed the S14 at (136.9, 122.6)
- removed the S14 at (272.8, 125.5)
- removed the S15 at (137.3, 103.6)
- removed the S15 at (272.5, 106.5)
- removed the S16 at (155.6, 141.9)
- removed the S16 at (254.1, 144.9)
- removed the S17 at (155.9, 122.9)
- removed the S17 at (253.8, 125.9)
- removed the S18 at (156.3, 103.9)
- removed the S18 at (253.5, 106.9)
- removed the S19 at (134.7, 163.6)
- removed the S19 at (275.0, 166.5)
- removed the S2 at (58.8, 137.8)
- removed the S2 at (350.9, 140.7)
- removed the S20 at (155.3, 165.6)
- removed the S20 at (254.4, 168.5)
- removed the S21 at (175.7, 172.0)
- removed the S21 at (234.1, 175.0)
- removed the S3 at (57.1, 118.9)
- removed the S3 at (352.6, 121.8)
- removed the S4 at (79.4, 155.1)
- removed the S4 at (330.4, 158.0)
- removed the S5 at (77.7, 136.2)
- removed the S5 at (332.0, 139.1)
- removed the S6 at (76.1, 117.2)
- removed the S6 at (333.7, 120.2)
- removed the S7 at (98.1, 142.9)
- removed the S7 at (311.6, 145.9)
- removed the S8 at (97.5, 124.0)
- removed the S8 at (312.2, 126.9)
- removed the S9 at (96.8, 105.0)
- removed the S9 at (312.9, 107.9)
- added S1: , keeb-footprints:Gateron-KS33+MX-Hotswap-1U, F.Cu at (112.0, 141.7)
- added S10: , keeb-footprints:Gateron-KS33+MX-Hotswap-1U, F.Cu at (168.4, 121.6)
- added S11: , keeb-footprints:Gateron-KS33+MX-Hotswap-1U, F.Cu at (167.7, 102.6)
- added S12: , keeb-footprints:Gateron-KS33+MX-Hotswap-1U, F.Cu at (167.1, 83.6)
- added S13: , keeb-footprints:Gateron-KS33+MX-Hotswap-1U, F.Cu at (188.0, 125.7)
- added S14: , keeb-footprints:Gateron-KS33+MX-Hotswap-1U, F.Cu at (188.4, 106.7)
- added S15: , keeb-footprints:Gateron-KS33+MX-Hotswap-1U, F.Cu at (188.7, 87.7)
- added S16: , keeb-footprints:Gateron-KS33+MX-Hotswap-1U, F.Cu at (207.0, 126.0)
- added S17: , keeb-footprints:Gateron-KS33+MX-Hotswap-1U, F.Cu at (207.4, 107.0)
- added S18: , keeb-footprints:Gateron-KS33+MX-Hotswap-1U, F.Cu at (207.7, 88.0)
- added S19: , keeb-footprints:Gateron-KS33+MX-Hotswap-1U, F.Cu at (186.2, 147.6)
- added S2: , keeb-footprints:Gateron-KS33+MX-Hotswap-1U, F.Cu at (110.3, 122.8)
- added S20: , keeb-footprints:Gateron-KS33+MX-Hotswap-1U, F.Cu at (206.8, 149.6)
- added S21: , keeb-footprints:Gateron-KS33+MX-Hotswap-1U, F.Cu at (227.1, 156.1)
- added S3: , keeb-footprints:Gateron-KS33+MX-Hotswap-1U, F.Cu at (108.7, 103.9)
- added S4: , keeb-footprints:Gateron-KS33+MX-Hotswap-1U, F.Cu at (130.9, 140.1)
- added S5: , keeb-footprints:Gateron-KS33+MX-Hotswap-1U, F.Cu at (129.2, 121.1)
- added S6: , keeb-footprints:Gateron-KS33-Hotswap+MX_Solderable_1U, F.Cu at (127.6, 102.2)
- added S7: , keeb-footprints:Gateron-KS33+MX-Hotswap-1U, F.Cu at (149.6, 127.0)
- added S8: , keeb-footprints:Gateron-KS33+MX-Hotswap-1U, F.Cu at (148.9, 108.0)
- added S9: , keeb-footprints:Gateron-KS33+MX-Hotswap-1U, F.Cu at (148.3, 89.0)
- REF**: moved to B.Cu
- moved REF** 53.3 mm to (126.7, 89.0), turned to 95 degrees

Commit message: made diode footprint, routed columns
Parts:
- added REF**: MountingHole_2.2mm_M2_DIN965_Pad, MountingHole:MountingHole_2.2mm_M2_DIN965_Pad, F.Cu at (138.4, 81.8)
- added REF**: DO-35_and_SOD-123, keeb-footprints:DO-35_and_SOD-123, F.Cu at (59.8, 117.2)
- SW1: renamed from S3; value (none) -> S
- SW10: renamed from S11; value (none) -> S
- SW11: renamed from S14; value (none) -> S
- SW12: renamed from S17; value (none) -> S
- SW13: renamed from S1; value (none) -> S
- SW14: renamed from S4; value (none) -> S
- SW15: renamed from S7; value (none) -> S
- SW16: renamed from S10; value (none) -> S
- SW17: renamed from S13; value (none) -> S
- SW18: renamed from S16; value (none) -> S
- SW19: renamed from S19; value (none) -> S
- SW2: renamed from S6; value (none) -> S
- SW20: renamed from S20; value (none) -> S
- SW21: renamed from S21; value (none) -> S
- SW3: renamed from S9; value (none) -> S
- SW4: renamed from S12; value (none) -> S
- SW5: renamed from S15; value (none) -> S
- SW6: renamed from S18; value (none) -> S
- SW7: renamed from S2; value (none) -> S
- SW8: renamed from S5; value (none) -> S
- SW9: renamed from S8; value (none) -> S
- turned SW1 to -175 degrees
- turned SW13 to -175 degrees
- turned SW7 to -175 degrees
Connections:
- SW1 pad 1: (no net) -> /LCol0
- SW1 pad 2: (no net) -> Net-(D1-A)
- SW10 pad 1: (no net) -> /LCol3
- SW10 pad 2: (no net) -> Net-(D10-A)
- SW11 pad 1: (no net) -> /LCol4
- SW11 pad 2: (no net) -> Net-(D11-A)
- SW12 pad 1: (no net) -> /LCol5
- SW12 pad 2: (no net) -> Net-(D12-A)
- SW13 pad 1: (no net) -> /LCol0
- SW13 pad 2: (no net) -> Net-(D13-A)
- SW14 pad 1: (no net) -> /LCol1
- SW14 pad 2: (no net) -> Net-(D14-A)
- SW15 pad 1: (no net) -> /LCol2
- SW15 pad 2: (no net) -> Net-(D15-A)
- SW16 pad 1: (no net) -> /LCol3
- SW16 pad 2: (no net) -> Net-(D16-A)
- SW17 pad 1: (no net) -> /LCol4
- SW17 pad 2: (no net) -> Net-(D17-A)
- SW18 pad 1: (no net) -> /LCol5
- SW18 pad 2: (no net) -> Net-(D18-A)
- SW19 pad 1: (no net) -> /LCol3
- SW19 pad 2: (no net) -> Net-(D19-A)
- SW2 pad 1: (no net) -> /LCol1
- SW2 pad 2: (no net) -> Net-(D2-A)
- SW20 pad 1: (no net) -> /LCol4
- SW20 pad 2: (no net) -> Net-(D20-A)
- SW21 pad 1: (no net) -> /LCol5
- SW21 pad 2: (no net) -> Net-(D21-A)
- SW3 pad 1: (no net) -> /LCol2
- SW3 pad 2: (no net) -> Net-(D3-A)
- SW4 pad 1: (no net) -> /LCol3
- SW4 pad 2: (no net) -> Net-(D4-A)
- SW5 pad 1: (no net) -> /LCol4
- SW5 pad 2: (no net) -> Net-(D5-A)
- SW6 pad 1: (no net) -> /LCol5
- SW6 pad 2: (no net) -> Net-(D6-A)
- SW7 pad 1: (no net) -> /LCol0
- SW7 pad 2: (no net) -> Net-(D7-A)
- SW8 pad 1: (no net) -> /LCol1
- SW8 pad 2: (no net) -> Net-(D8-A)
- SW9 pad 1: (no net) -> /LCol2
- SW9 pad 2: (no net) -> Net-(D9-A)
Routing:
- net /LCol1: track 0.00 -> 60.0 mm
- net /LCol0: track 0.00 -> 46.9 mm
- net /LCol4: track 0.00 -> 46.4 mm
- net /LCol5: track 0.00 -> 46.4 mm
- net /LCol2: track 0.00 -> 46.3 mm
- net /LCol3: track 0.00 -> 46.3 mm
- net Net-(D2-A): track 0.00 -> 12.0 mm
- net Net-(D13-A): track 0.00 -> 11.2 mm
- net Net-(D8-A): track 0.00 -> 11.2 mm
- net Net-(D14-A): track 0.00 -> 11.2 mm
- net Net-(D7-A): track 0.00 -> 11.2 mm
- net Net-(D1-A): track 0.00 -> 11.2 mm
