File: PCB/praevius.kicad_sch (KiCad schematic)
At the start: 0 parts

Commit message: Started schematic
Parts:
- added D1, D10, D11, D12, D13, D14, D15, D16, D17, D18, D19, D2, D20, D21, D22, D23, D24, D25, D26, D27, D28, D29, D3, D30, D31, D32, D33, D34, D35, D36, D37, D38, D39, D4, D43, D44, D45, D5, D6, D7, D8, D9: 1N4149, Diode_THT:D_DO-35_SOD27_P7.62mm_Horizontal, symbol Diode:1N4149
- added MCU1, MCU2: XIAO-nRF52840-Plus-SMD, Seeed_Studio_XIAO_Series:XIAO-nRF52840-Plus-SMD, symbol Seeed_Studio_XIAO_Series:XIAO-nRF52840_Plus_SMD
- added SW1, SW10, SW11, SW12, SW13, SW14, SW15, SW16, SW17, SW18, SW19, SW2, SW20, SW21, SW3, SW4, SW5, SW6, SW7, SW8, SW9: SW_Push_45deg, symbol Switch:SW_Push_45deg
- added SW22, SW23, SW24, SW25, SW26, SW27, SW28, SW29, SW30, SW31, SW32, SW33, SW34, SW35, SW36, SW37, SW38, SW39, SW43, SW44, SW45: SW_Push_45deg, Button_Switch_SMD:Nidec_Copal_CAS-120A, symbol Switch:SW_Push_45deg
Connections:
- new net: D24.2 (A), SW24.1
- new net: D9.2 (A), SW9.2
- new net: D27.2 (A), SW27.1
- new net: D2.2 (A), SW2.2
- new net: D35.2 (A), SW35.1
- new net: D17.2 (A), SW17.2
- new net: D4.2 (A), SW4.2
- new net: D43.2 (A), SW43.1
- new net: D30.2 (A), SW30.1
- new net: D22.2 (A), SW22.1
- new net: D5.2 (A), SW5.2
- new net: D8.2 (A), SW8.2
- new net: D11.2 (A), SW11.2
- new net: D7.2 (A), SW7.2
- new net: D3.2 (A), SW3.2
- new net: D29.2 (A), SW29.1
- new net: D21.2 (A), SW21.2
- new net: D13.2 (A), SW13.2
- new net: D36.2 (A), SW36.1
- new net: D37.2 (A), SW37.1
- new net: D31.2 (A), SW31.1
- new net: D20.2 (A), SW20.2
- new net: D12.2 (A), SW12.2
- new net: D26.2 (A), SW26.1
- new net: D44.2 (A), SW44.1
- new net: D39.2 (A), SW39.1
- new net: D28.2 (A), SW28.1
- new net: D45.2 (A), SW45.1
- new net: D19.2 (A), SW19.2
- new net: D34.2 (A), SW34.1
- new net: D18.2 (A), SW18.2
- new net: D15.2 (A), SW15.2
- new net: D32.2 (A), SW32.1
- new net: D1.2 (A), SW1.2
- new net: D6.2 (A), SW6.2
- new net: D16.2 (A), SW16.2
- new net: D23.2 (A), SW23.1
- new net: D33.2 (A), SW33.1
- new net: D38.2 (A), SW38.1
- new net: D25.2 (A), SW25.1
- new net: D14.2 (A), SW14.2
- new net: D10.2 (A), SW10.2
- new net LCol0: SW1.1, SW13.1, SW7.1
- new net LCol1: SW14.1, SW2.1, SW8.1
- new net LCol2: SW15.1, SW3.1, SW9.1
- new net LCol3: SW10.1, SW16.1, SW19.1, SW4.1
- new net LCol4: SW11.1, SW17.1, SW20.1, SW5.1
- new net LCol5: SW12.1, SW18.1, SW21.1, SW6.1
- new net LRow0: D1.1 (K), D2.1 (K), D3.1 (K), D4.1 (K), D5.1 (K), D6.1 (K)
- new net LRow1: D10.1 (K), D11.1 (K), D12.1 (K), D7.1 (K), D8.1 (K), D9.1 (K)
- new net LRow2: D13.1 (K), D14.1 (K), D15.1 (K), D16.1 (K), D17.1 (K), D18.1 (K)
- new net LRow3: D19.1 (K), D20.1 (K), D21.1 (K)
- new net RCol0: SW27.2, SW33.2, SW39.2
- new net RCol1: SW26.2, SW32.2, SW38.2
- new net RCol2: SW25.2, SW31.2, SW37.2
- new net RCol3: SW24.2, SW30.2, SW36.2, SW45.2
- new net RCol4: SW23.2, SW29.2, SW35.2, SW44.2
- new net RCol5: SW22.2, SW28.2, SW34.2, SW43.2
- new net RRow0: D22.1 (K), D23.1 (K), D24.1 (K), D25.1 (K), D26.1 (K), D27.1 (K)
- new net RRow1: D28.1 (K), D29.1 (K), D30.1 (K), D31.1 (K), D32.1 (K), D33.1 (K)
- new net RRow2: D34.1 (K), D35.1 (K), D36.1 (K), D37.1 (K), D38.1 (K), D39.1 (K)
- new net RRow3: D43.1 (K), D44.1 (K), D45.1 (K)

Commit message: made diode footprint, routed columns
Parts:
- D1, D10, D2, D3, D4, D5, D6, D7, D8, D9: footprint Diode_THT:D_DO-35_SOD27_P7.62mm_Horizontal -> keeb-footprints:DO-35_and_SOD-123
- D11, D12, D13, D14, D15, D16, D17, D18, D19, D20, D21, D22, D23, D24, D25, D26, D27, D28, D29, D30, D31, D32, D33, D34, D35, D36, D37, D38, D39, D43, D44, D45: footprint Diode_THT:D_DO-35_SOD27_P7.62mm_Horizontal -> (none)
- SW1, SW10, SW11, SW12, SW13, SW14, SW15, SW16, SW17, SW18, SW19, SW20, SW21, SW3, SW4, SW5, SW6, SW7, SW8, SW9: value SW_Push_45deg -> S; footprint (none) -> keeb-footprints:Gateron-KS33+MX-Hotswap-1U
- SW2: value SW_Push_45deg -> S; footprint (none) -> keeb-footprints:Gateron-KS33-Hotswap+MX_Solderable_1U
- SW22, SW23, SW24, SW25, SW26, SW27, SW28, SW29, SW30, SW31, SW32, SW33, SW34, SW35, SW36, SW37, SW38, SW39, SW43, SW44, SW45: value SW_Push_45deg -> S; footprint Button_Switch_SMD:Nidec_Copal_CAS-120A -> (none)
