File: PCB/_restore_backup_2026-10-10T09-29-51-118/praevius.kicad_pcb (KiCad board)
At the start: 2 copper layers, 32 x 19 mm, 44 parts, among them SW1 S, SW10 S, SW11 S, SW12 S, SW13 S, SW14 S, SW15 S, SW16 S, SW17 S, SW18 S, SW19 S, SW2 S, SW20 S, SW21 S, SW3 S, SW4 S, SW5 S, SW6 S, SW7 S, SW8 S, SW9 S

Commit message: edited diode footprint, routed, research trackpad
Parts:
- removed the REF** at (48.7, 141.9)
- added ?: , , F.Cu at (121.7, 142.8)
- moved D15 19.1 mm to (153.7, 136.4)
Routing:
- net /LRow2: track 91.4 -> 114.4 mm
- net /LRow0: track 93.5 -> 112.7 mm
- net /LRow1: track 90.2 -> 109.4 mm
- net Net-(D15-A): track 33.4 -> 15.8 mm
Other:
- board outline removed
